File: ameoba.kicad_pcb (KiCad board)
At the start: 2 copper layers, 18.7 x 17.7 mm, 23 parts

Commit message: update
Parts:
- moved G_logo 0.91 mm to (21.8, 22.0)
- moved ? 0.28 mm to (30.2, 17.4)
- renumbered G*** to G_logo
Changed lines of the file:
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@@
       (outputformat 1)
       (mirror false)
-      (drillshape 1)
+      (drillshape 0)
       (scaleselection 1)
-      (outputdirectory "")
+      (outputdirectory "Gerber/")
     )
   )
@@
   )
   (footprint "" (layer "F.Cu")
-    (at 30.206577 17.675453)
+    (at 30.206577 17.4)
     (fp_text reference "" (at 0 0) (layer "F.SilkS")
       (effects (font (size 1.27 1.27) (thickness 0.15)))
@@
       (effects (font (size 1.27 1.27) (thickness 0.15)))
     )
-    (pad "1" thru_hole rect (at -0.065901 0.058587) (size 1 1) (drill 0.6) (layers *.Cu *.Mask)
+    (pad "1" thru_hole rect (at -0.065901 -0.212363) (size 1 1) (drill 0.6) (layers *.Cu *.Mask)
       (net 4 "GND") (pinfunction "Pin_1") (pintype "passive"))
   )
@@
   )
   (footprint "LOGO" (layer "F.Cu")
-    (at 21.089681 21.4544)
+    (at 21.808912 22.010282)
     (attr board_only exclude_from_pos_files exclude_from_bom)
-    (fp_text reference "G***" (at 0 0) (layer "F.SilkS") hide
+    (fp_text reference "G_logo" (at 0 0) (layer "F.SilkS") hide
       (effects (font (size 1.524 1.524) (thickness 0.3)))
     )
@@
     (fp_arc (start -1.655353 1.637847) (mid -1.773397 1.588075) (end -1.831183 1.47374) (layer "Edge.Cuts") (width 0.12))
     (fp_arc (start -1.83223 -1.451854) (mid -1.782457 -1.569897) (end -1.668123 -1.627684) (layer "Edge.Cuts") (width 0.12))
-    (fp_arc (start 1.656019 -1.628728) (mid 1.774062 -1.578955) (end 1.831849 -1.464621) (layer "Edge.Cuts") (width 0.12))
-    (fp_arc (start 1.844615 1.472697) (mid 1.794842 1.59074) (end 1.680508 1.648527) (layer "Edge.Cuts") (width 0.12))
+    (fp_arc (start 1.656019 -1.628728) (mid 1.774063 -1.578955) (end 1.831849 -1.464621) (layer "Edge.Cuts") (width 0.12))
+    (fp_arc (start 1.844615 1.472697) (mid 1.794841 1.590738) (end 1.680508 1.648527) (layer "Edge.Cuts") (width 0.12))
     (pad "1" smd rect locked (at -2.653636 -0.747946 180) (size 1.492724 0.824104) (layers "B.Cu" "B.Paste" "B.Mask")
       (net 5 "VCC"))
